File: hardware/OpenLog.brd (EAGLE design)
At the start: 15.2 x 19.1 mm, 26 parts, among them Q1 16MHZ, U1 ATMEGA328P_TQFP, U2 3.3V MIC5205, U3 microSD Socket

Commit message: Swapped resistor on grn LED to 330 for better visibility
Parts:
- R6: value 1K -> 330
Changed lines of the file:
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@@
 <?xml version="1.0" encoding="utf-8"?>
 <!DOCTYPE eagle SYSTEM "eagle.dtd">
-<eagle version="7.2.0">
+<eagle version="7.3.0">
 <drawing>
 <settings>
@@
 <attribute name="PROD_ID" value="CAP-00810" x="1.27" y="11.43" size="1.778" layer="27" rot="R270" display="off"/>
 </element>
-<element name="R6" library="SparkFun-Resistors" package="0603-RES" value="1K" x="1.844040625" y="14.4500625" smashed="yes" rot="R180">
+<element name="R6" library="SparkFun-Resistors" package="0603-RES" value="330" x="1.844040625" y="14.4500625" smashed="yes" rot="R180">
 <attribute name="NAME" x="3.844040625" y="14.4500625" size="1.27" layer="25"/>
-<attribute name="VALUE" value="1K" x="1.501640625" y="15.0850625" size="0.4064" layer="27"/>
-<attribute name="PROD_ID" value="RES-07856" x="1.844040625" y="14.4500625" size="1.778" layer="27" rot="R180" display="off"/>
+<attribute name="VALUE" value="330" x="1.501640625" y="15.0850625" size="0.4064" layer="27"/>
+<attribute name="PROD_ID" value="RES-00818" x="1.844040625" y="14.4500625" size="1.778" layer="27" rot="R180" display="off"/>
 </element>
 <element name="D3" library="SparkFun-LED" package="LED-0603" value="GREEN" x="1.86181875" y="15.814040625" smashed="yes" rot="R270">
